Commit message: two mani motion planning with 6+6,12 dof

File: curobo/robots/piper/piper_arm.urdf (robot description, URDF)
Before this commit: robot piper_v100_arm, 8 links, 7 joints
Links:
- link gripper_center: geometry collision sphere radius=0.055

Commit message: add rail mounted piper simulation

File: curobo/robots/piper/piper_arm.urdf (robot description, URDF)
Before this commit: robot piper_v100_arm, 8 links, 7 joints
Links:
- added link gripper_body
- added link gripper_contact
- link gripper_center: geometry 
Joints:
- added joint gripper_center_to_body: type fixed, parent gripper_center, child gripper_body, origin xyz=0 0 0 rpy=0 0 0
- added joint gripper_center_to_contact: type fixed, parent gripper_center, child gripper_contact, origin xyz=0 0 0 rpy=0 0 0
